File: hardware/rev_a/embedded-gw.sch (EAGLE design)
At the start: 42 parts, among them J1 DM3BT-DSF-PEJS, J2 USB-A-MALE-PLUG, J3 TC2030-JLINK-NL, U1 ESP32-WROVER-E, U2 ESP32-WROVER-E, U3 AP7362A-33SP-13, U4 BC840M, U5 CP2102N-20, U6 ESDR0502N

Commit message: forgot to save
Connections:
- removed net VSPIHD: U1.IO21
- removed net VSPIWP: U1.IO22
Changed lines of the file:
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@@
 <grid distance="0.1" unitdist="inch" unit="inch" style="lines" multiple="1" display="no" altdistance="0.01" altunitdist="inch" altunit="inch"/>
 <layers>
-<layer number="1" name="Top" color="4" fill="1" visible="yes" active="no"/>
-<layer number="2" name="Route2" color="16" fill="1" visible="yes" active="no"/>
-<layer number="3" name="Route3" color="17" fill="1" visible="yes" active="no"/>
-<layer number="4" name="Route4" color="18" fill="1" visible="yes" active="no"/>
-<layer number="5" name="Route5" color="19" fill="1" visible="yes" active="no"/>
-<layer number="6" name="Route6" color="25" fill="1" visible="yes" active="no"/>
-<layer number="7" name="Route7" color="26" fill="1" visible="yes" active="no"/>
-<layer number="8" name="Route8" color="27" fill="1" visible="yes" active="no"/>
-<layer number="9" name="Route9" color="28" fill="1" visible="yes" active="no"/>
-<layer number="10" name="Route10" color="29" fill="1" visible="yes" active="no"/>
-<layer number="11" name="Route11" color="30" fill="1" visible="yes" active="no"/>
-<layer number="12" name="Route12" color="20" fill="1" visible="yes" active="no"/>
-<layer number="13" name="Route13" color="21" fill="1" visible="yes" active="no"/>
-<layer number="14" name="Route14" color="22" fill="1" visible="yes" active="no"/>
-<layer number="15" name="Route15" color="23" fill="1" visible="yes" active="no"/>
-<layer number="16" name="Bottom" color="1" fill="1" visible="yes" active="no"/>
-<layer number="17" name="Pads" color="2" fill="1" visible="yes" active="no"/>
-<layer number="18" name="Vias" color="2" fill="1" visible="yes" active="no"/>
-<layer number="19" name="Unrouted" color="6" fill="1" visible="yes" active="no"/>
-<layer number="20" name="Dimension" color="24" fill="1" visible="yes" active="no"/>
-<layer number="21" name="tPlace" color="7" fill="1" visible="yes" active="no"/>
-<layer number="22" name="bPlace" color="7" fill="1" visible="yes" active="no"/>
-<layer number="23" name="tOrigins" color="15" fill="1" visible="yes" active="no"/>
-<layer number="24" name="bOrigins" color="15" fill="1" visible="yes" active="no"/>
-<layer number="25" name="tNames" color="7" fill="1" visible="yes" active="no"/>
-<layer number="26" name="bNames" color="7" fill="1" visible="yes" active="no"/>
-<layer number="27" name="tValues" color="7" fill="1" visible="yes" active="no"/>
-<layer number="28" name="bValues" color="7" fill="1" visible="yes" active="no"/>
+<layer number="1" name="Top" color="4" fill="1" visible="no" active="no"/>
+<layer number="2" name="Route2" color="16" fill="1" visible="no" active="no"/>
+<layer number="3" name="Route3" color="17" fill="1" visible="no" active="no"/>
+<layer number="4" name="Route4" color="18" fill="1" visible="no" active="no"/>
+<layer number="5" name="Route5" color="19" fill="1" visible="no" active="no"/>
+<layer number="6" name="Route6" color="25" fill="1" visible="no" active="no"/>
+<layer number="7" name="Route7" color="26" fill="1" visible="no" active="no"/>
+<layer number="8" name="Route8" color="27" fill="1" visible="no" active="no"/>
+<layer number="9" name="Route9" color="28" fill="1" visible="no" active="no"/>
+<layer number="10" name="Route10" color="29" fill="1" visible="no" active="no"/>
+<layer number="11" name="Route11" color="30" fill="1" visible="no" active="no"/>
+<layer number="12" name="Route12" color="20" fill="1" visible="no" active="no"/>
+<layer number="13" name="Route13" color="21" fill="1" visible="no" active="no"/>
+<layer number="14" name="Route14" color="22" fill="1" visible="no" active="no"/>
+<layer number="15" name="Route15" color="23" fill="1" visible="no" active="no"/>
+<layer number="16" name="Bottom" color="1" fill="1" visible="no" active="no"/>
+<layer number="17" name="Pads" color="2" fill="1" visible="no" active="no"/>
+<layer number="18" name="Vias" color="2" fill="1" visible="no" active="no"/>
+<layer number="19" name="Unrouted" color="6" fill="1" visible="no" active="no"/>
+<layer number="20" name="Dimension" color="24" fill="1" visible="no" active="no"/>
+<layer number="21" name="tPlace" color="7" fill="1" visible="no" active="no"/>
+<layer number="22" name="bPlace" color="7" fill="1" visible="no" active="no"/>
+<layer number="23" name="tOrigins" color="15" fill="1" visible="no" active="no"/>
+<layer number="24" name="bOrigins" color="15" fill="1" visible="no" active="no"/>
+<layer number="25" name="tNames" color="7" fill="1" visible="no" active="no"/>
+<layer number="26" name="bNames" color="7" fill="1" visible="no" active="no"/>
+<layer number="27" name="tValues" color="7" fill="1" visible="no" active="no"/>
+<layer number="28" name="bValues" color="7" fill="1" visible="no" active="no"/>
 <layer number="29" name="tStop" color="7" fill="3" visible="no" active="no"/>
 <layer number="30" name="bStop" color="7" fill="6" visible="no" active="no"/>
@@
 <layer number="35" name="tGlue" color="7" fill="4" visible="no" active="no"/>
 <layer number="36" name="bGlue" color="7" fill="5" visible="no" active="no"/>
-<layer number="37" name="tTest" color="7" fill="1" visible="yes" active="no"/>
-<layer number="38" name="bTest" color="7" fill="1" visible="yes" active="no"/>
+<layer number="37" name="tTest" color="7" fill="1" visible="no" active="no"/>
+<layer number="38" name="bTest" color="7" fill="1" visible="no" active="no"/>
 <layer number="39" name="tKeepout" color="4" fill="11" visible="no" active="no"/>
 <layer number="40" name="bKeepout" color="1" fill="11" visible="no" active="no"/>
@@
 <layer number="44" name="Drills" color="7" fill="1" visible="no" active="no"/>
 <layer number="45" name="Holes" color="7" fill="1" visible="no" active="no"/>
-<layer number="46" name="Milling" color="3" fill="1" visible="yes" active="no"/>
-<layer number="47" name="Measures" color="7" fill="1" visible="yes" active="no"/>
-<layer number="48" name="Document" color="7" fill="1" visible="yes" active="no"/>
-<layer number="49" name="Reference" color="7" fill="1" visible="yes" active="no"/>
-<layer number="50" name="dxf" color="7" fill="1" visible="yes" active="no"/>
-<layer number="51" name="tDocu" color="7" fill="1" visible="yes" active="no"/>
-<layer number="52" name="bDocu" color="7" fill="1" visible="yes" active="no"/>
-<layer number="53" name="tGND_GNDA" color="7" fill="9" visible="yes" active="no"/>
-<layer number="54" name="bGND_GNDA" color="1" fill="9" visible="yes" active="no"/>
-<layer number="56" name="wert" color="7" fill="1" visible="yes" active="no"/>
-<layer number="57" name="tCAD" color="7" fill="1" visible="yes" active="no"/>
-<layer number="59" name="Invisible" color="7" fill="1" visible="yes" active="no"/>
-<layer number="60" name="bCarbon" color="7" fill="1" visible="yes" active="no"/>
-<layer number="61" name="stand" color="7" fill="1" visible="yes" active="no"/>
+<layer number="46" name="Milling" color="3" fill="1" visible="no" active="no"/>
+<layer number="47" name="Measures" color="7" fill="1" visible="no" active="no"/>
+<layer number="48" name="Document" color="7" fill="1" visible="no" active="no"/>
+<layer number="49" name="Reference" color="7" fill="1" visible="no" active="no"/>
+<layer number="50" name="dxf" color="7" fill="1" visible="no" active="no"/>
+<layer number="51" name="tDocu" color="7" fill="1" visible="no" active="no"/>
+<layer number="52" name="bDocu" color="7" fill="1" visible="no" active="no"/>
+<layer number="53" name="tGND_GNDA" color="7" fill="9" visible="no" active="no"/>
+<layer number="54" name="bGND_GNDA" color="1" fill="9" visible="no" active="no"/>
+<layer number="56" name="wert" color="7" fill="1" visible="no" active="no"/>
+<layer number="57" name="tCAD" color="7" fill="1" visible="no" active="no"/>
+<layer number="59" name="Invisible" color="7" fill="1" visible="no" active="no"/>
+<layer number="60" name="bCarbon" color="7" fill="1" visible="no" active="no"/>
+<layer number="61" name="stand" color="7" fill="1" visible="no" active="no"/>
 <layer number="88" name="SimResults" color="9" fill="1" visible="yes" active="yes"/>
 <layer number="89" name="SimProbes" color="9" fill="1" visible="yes" active="yes"/>
@@
 </segment>
 </net>
-<net name="VSPIWP" class="0">
-<segment>
-<pinref part="U1" gate="G$1" pin="IO22"/>
-<wire x1="91.44" y1="147.32" x2="93.98" y2="147.32" width="0.1524" layer="91"/>
-<label x="93.98" y="147.32" size="1.27" layer="95" xref="yes"/>
-</segment>
-</net>
-<net name="VSPIHD" class="0">
-<segment>
-<pinref part="U1" gate="G$1" pin="IO21"/>
-<wire x1="91.44" y1="144.78" x2="93.98" y2="144.78" width="0.1524" layer="91"/>
-<label x="93.98" y="144.78" size="1.27" layer="95" xref="yes"/>
-</segment>
-</net>

Commit message: start layout
Parts:
- removed U4: BC840M, chips:BC840M
- added C12, C13: 12pF, passives:CAPACITOR0402_CAP
- added R10, R8: 10k, passives:RESISTOR0402_RES
- added U7: BT840X, BT840X:BT840X
- added X1: ABS05-32.768KHZ-9-T, crystals:ABS05-32.768KHZ-9-T
- C5, C6, C7: device passives:CAPACITOR0402_CAP -> passives:CAPACITOR0805_CAP
- D3: value BLUE -> YELLOW; DIGIKEY 160-1827-1-ND -> 160-1831-1-ND; MPN LTST-C193TBKT-5A -> LTST-C193KSKT-5A
- D4, D7: value YELLOW -> BLUE; DIGIKEY 160-1831-1-ND -> 160-1827-1-ND; MPN LTST-C193KSKT-5A -> LTST-C193TBKT-5A
- D5: value BLUE -> RED; DIGIKEY 160-1827-1-ND -> 160-1830-1-ND; MPN LTST-C193TBKT-5A -> LTST-C193KRKT-5A
- D6: value RED -> YELLOW; DIGIKEY 160-1830-1-ND -> 160-1831-1-ND; MPN LTST-C193KRKT-5A -> LTST-C193KSKT-5A
- renumbered D11 to D9, D12 to D10
Connections:
- net N$1 renamed RXD
- net N$2 renamed TXD
- net N$3 renamed VBUS
- net N$4 renamed D+
- net N$5 renamed D-
- removed net ESP32_MISO: U1.IO19, U2.IO19
- removed net ESP32_MOSI: U1.IO23, U2.IO23
- removed net ESP32_SCLK: U1.IO18, U2.IO18
- removed net NRF_HANDSHAKE: U2.IO25, U4.A0/P101
- new net ESP32_0_ID: R8.2, U1.IO26
- new net ESP32_1_ID: R10.1, U2.IO26
- new net N$1: U7.VBUS
- new net N$2: C12.2, U7.P0.00/XL1, X1.2
- new net N$3: C13.2, U7.P0.01/XL2, X1.1
- net !RESET: now also U7.P0.18/RESET; no longer U4.B4/P018/RESET
- net !SD_INSERTED: now also U1.IO27, U2.IO27
- net ESP32_CS: now also U1.IO25, U2.IO25; no longer U1.IO5, U2.IO5
- net GND: now also C12.1, C13.1, R8.1, U7.GND; no longer U4.G0/VSS, U4.G4/VSS, U4.G5/VSS, U4.G6/VSS, U4.H4/VSS, U4.H5/VSS, U4.H6/VSS, U4.H7/VSS
- net LED10: no longer R11.2
- net LED11: no longer R12.2
- net LED12: no longer R13.2
- net N$14: now also D3.CATHODE; no longer D4.CATHODE
- net N$15: now also D4.CATHODE; no longer D3.CATHODE
- net N$19: now also D5.CATHODE; no longer D6.CATHODE
- net N$20: now also D6.CATHODE; no longer D7.CATHODE
- net N$21: now also D7.CATHODE; no longer D5.CATHODE
- net NRF_CS: now also U1.IO5, U2.IO5, U7.P0.20; no longer U2.IO13, U4.A1/P025
- net NRF_LED0: now also R11.2, U7.P0.13; no longer U4.E5/P031
- net NRF_LED1: now also R12.2, U7.P0.14; no longer U4.E6/P026
- net NRF_LED2: now also R13.2, U7.P0.15; no longer U4.E7/P004
- net NRF_MISO: now also U1.IO19, U2.IO19, U7.P0.21; no longer U2.IO2, U4.C6/P109
- net NRF_MOSI: now also U1.IO23, U2.IO23, U7.P0.22; no longer U2.IO15, U4.C7/P008
- net NRF_SCLK: now also U1.IO18, U2.IO18, U7.P0.19; no longer U2.IO14, U4.B7/P012
- net SD_HOST_CLK: now also U2.IO14
- net SD_HOST_CMD: now also U2.IO15
- net SD_HOST_D0: now also U2.IO2
- net SD_HOST_D1: now also U2.IO4
- net SD_HOST_D2: now also U2.IO12
- net SD_HOST_D3: now also U2.IO13
- net SWDCLK: now also U7.SWCLK; no longer U4.C1/SWDCLK
- net SWDIO: now also U7.SWDIO; no longer U4.B1/SWDIO
- net VCC: now also R10.2, U7.VDD, U7.VDDH; no longer U4.A7/VDDH, U4.F5/VDD
Other:
- moved on the sheet: C10, C11, C5, C6, D3, D4, D5, D6, D7, U3

Commit message: Clean up and run the script
rename parts, clean up bom, cam, package up
Parts:
- removed U7: BT840X, BT840X:BT840X
- added D11: BLUE, leds:LED0603
- added U4: ESDR0502N, chips:ESDR0502N
- C1: value 1.0uF -> 12pF; DIGIKEY 1276-1010-1-ND -> 490-GCM1555C1H120GA16DCT-ND; MPN CL05A105KQ5NNNC -> GCM1555C1H120GA16D
- C10: value 1.0uF -> 4.7uF; device passives:CAPACITOR0402_CAP -> passives:CAPACITOR0603_CAP; DIGIKEY 1276-1010-1-ND -> 1276-1045-1-ND; MPN CL05A105KQ5NNNC -> CL10A475KQ8NNNC
- C11: value 0.1uF -> 10uF; device passives:CAPACITOR0402_CAP -> passives:CAPACITOR0805_CAP; DIGIKEY 1276-1511-1-ND -> 1276-2404-1-ND; MPN CL05B104KQ5NNNC -> CL21A106KQCLNNC
- C12, C13: value 12pF -> 10uF; device passives:CAPACITOR0402_CAP -> passives:CAPACITOR0805_CAP; DIGIKEY 490-GCM1555C1H120GA16DCT-ND -> 1276-2404-1-ND; MPN GCM1555C1H120GA16D -> CL21A106KQCLNNC
- C2: value 0.1uF -> 12pF; DIGIKEY 1276-1511-1-ND -> 490-GCM1555C1H120GA16DCT-ND; MPN CL05B104KQ5NNNC -> GCM1555C1H120GA16D
- C3: value 4.7uF -> 0.1uF; device passives:CAPACITOR0603_CAP -> passives:CAPACITOR0402_CAP; DIGIKEY 1276-1045-1-ND -> 1276-1511-1-ND; MPN CL10A475KQ8NNNC -> CL05B104KQ5NNNC
- C5, C6: value 10uF -> 0.1uF; device passives:CAPACITOR0805_CAP -> passives:CAPACITOR0402_CAP; DIGIKEY 1276-2404-1-ND -> 1276-1511-1-ND; MPN CL21A106KQCLNNC -> CL05B104KQ5NNNC
- C7: value 10uF -> 1.0uF; device passives:CAPACITOR0805_CAP -> passives:CAPACITOR0402_CAP; DIGIKEY 1276-2404-1-ND -> 1276-1010-1-ND; MPN CL21A106KQCLNNC -> CL05A105KQ5NNNC
- C9: value 0.1uF -> 1.0uF; DIGIKEY 1276-1511-1-ND -> 1276-1010-1-ND; MPN CL05B104KQ5NNNC -> CL05A105KQ5NNNC
- D1: value EMIF06-MSD01F2 -> (none); device passives:EMIF06-MSD01F2 -> passives:DIODE_ZENER0201; DIGIKEY (none) -> ESD7381MUT5GOSCT-ND; MPN (none) -> ESD7381MUT5G
- D10, D4: value BLUE -> YELLOW; DIGIKEY 160-1827-1-ND -> 160-1831-1-ND; MPN LTST-C193TBKT-5A -> LTST-C193KSKT-5A
- D2: value RED -> EMIF06-MSD01F2; device leds:LED0603 -> passives:EMIF06-MSD01F2; DIGIKEY 160-1830-1-ND -> (none); MPN LTST-C193KRKT-5A -> (none)
- D3, D9: value YELLOW -> RED; DIGIKEY 160-1831-1-ND -> 160-1830-1-ND; MPN LTST-C193KSKT-5A -> LTST-C193KRKT-5A
- D8: value RED -> BLUE; DIGIKEY 160-1830-1-ND -> 160-1827-1-ND; MPN LTST-C193KRKT-5A -> LTST-C193TBKT-5A
- J2: value USB-A-MALE-PLUG -> TC2030-JLINK-NL; device connector:USB-A-MALE-PLUG -> connector:TC2030-JLINK-NL
- J3: value TC2030-JLINK-NL -> USB-A-MALE-PLUG; device connector:TC2030-JLINK-NL -> connector:USB-A-MALE-PLUG
- R1: value 10k -> 100; DIGIKEY RMCF0402JT10K0CT-ND -> 311-100JRCT-ND; MPN RMCF0402JT10K0 -> RC0402JR-07100RL
- R11, R12: value 470 -> 10k; DIGIKEY 311-470LRCT-ND -> RMCF0402JT10K0CT-ND; MPN RC0402FR-07470RL -> RMCF0402JT10K0
- R13: value 100 -> 10k; DIGIKEY 311-100JRCT-ND -> RMCF0402JT10K0CT-ND; MPN RC0402JR-07100RL -> RMCF0402JT10K0
- R2: value 470 -> 100; DIGIKEY 311-470LRCT-ND -> 311-100JRCT-ND; MPN RC0402FR-07470RL -> RC0402JR-07100RL
- R7: value 100 -> 470; DIGIKEY 311-100JRCT-ND -> 311-470LRCT-ND; MPN RC0402JR-07100RL -> RC0402FR-07470RL
- R8, R9: value 10k -> 470; DIGIKEY RMCF0402JT10K0CT-ND -> 311-470LRCT-ND; MPN RMCF0402JT10K0 -> RC0402FR-07470RL
- U1: value ESP32-WROVER-E -> AP7362A-33SP-13; device chips:ESP32-WROVER-E -> chips:AP7362A-33SP-13
- U2: value ESP32-WROVER-E -> BT840X; device chips:ESP32-WROVER-E -> BT840X:BT840X
- U3: value AP7362A-33SP-13 -> CP2102N-20; device chips:AP7362A-33SP-13 -> chips:CP2102N-20
- U5: value CP2102N-20 -> ESP32-WROVER-E; device chips:CP2102N-20 -> chips:ESP32-WROVER-E
- U6: value ESDR0502N -> ESP32-WROVER-E; device chips:ESDR0502N -> chips:ESP32-WROVER-E
Connections:
- removed net N$1: U7.VBUS
- removed net N$12 (its old number): D2.CATHODE, R2.1
- new net N$14: D4.CATHODE, R5.1
- new net NC: U2.VBUS
- net !RESET: now also J2.!RESET, U2.P0.18/RESET; no longer J3.!RESET, U7.P0.18/RESET
- net !SD_INSERTED: now also D1.CATHODE, R11.2, U5.IO27, U6.IO27; no longer R9.2, U1.IO27, U2.IO27
- net D+: now also J3.D+, U3.D+, U4.D+; no longer J2.D+, U5.D+, U6.D+
- net D-: now also J3.D-, U3.D-, U4.D-; no longer J2.D-, U5.D-, U6.D-
- net ESP32_0_ID: now also R12.2, U5.IO26; no longer R8.2, U1.IO26
- net ESP32_0_RXD: now also U5.RXD0; no longer U1.RXD0
- net ESP32_0_TXD: now also U5.TXD0; no longer U1.TXD0
- net ESP32_1_ID: now also R13.1, U6.IO26; no longer R10.1, U2.IO26
- net ESP32_1_RXD: now also U6.RXD0; no longer U2.RXD0
- net ESP32_1_TXD: now also U6.TXD0; no longer U2.TXD0
- net ESP32_CS: now also U5.IO25, U6.IO25; no longer U1.IO25, U2.IO25
- net ESP32_HANDSHAKE: now also U5.IO33, U6.IO33; no longer U1.IO33, U2.IO33
- net GND: now also C1.1, C12.2, C13.2, C2.1, D1.ANODE, D2.VSS, R12.1, U4.GND; no longer C1.2, C12.1, C13.1, C2.2, D1.VSS, R8.1, U7.GND
- net LED00: now also R4.2, U5.IO34; no longer R2.2, U1.IO34
- net LED01: now also R5.2, U5.IO35; no longer R4.2, U1.IO35
- net LED02: now also R1.2, U5.IO32; no longer R3.2, U1.IO32
- net LED10: now also R6.2, U6.IO34; no longer R5.2, U2.IO34
- net LED11: now also R7.2, U6.IO35; no longer R6.2, U2.IO35
- net LED12: now also R2.2, U6.IO32; no longer R7.2, U2.IO32
- net N$10: now also D2.SD_DAT2; no longer D1.SD_DAT2
- net N$11: now also D2.SD_DAT3; no longer D1.SD_DAT3
- net N$13: now also D2.SD_CLK; no longer D1.SD_CLK
- net N$15: now also D7.CATHODE, R1.1; no longer D4.CATHODE, R3.1
- net N$19: now also R6.1; no longer R5.1
- net N$2: now also C1.2, U2.P0.00/XL1; no longer C12.2, U7.P0.00/XL1
- net N$20: now also R7.1; no longer R6.1
- net N$21: now also D8.CATHODE, R2.1; no longer D7.CATHODE, R7.1
- net N$22: now also D9.CATHODE, R8.1; no longer D8.CATHODE, R11.1
- net N$23: now also D10.CATHODE, R9.1; no longer D9.CATHODE, R12.1
- net N$24: now also D11.CATHODE, R3.1; no longer D10.CATHODE, R13.1
- net N$3: now also C2.2, U2.P0.01/XL2; no longer C13.2, U7.P0.01/XL2
- net N$6: now also D2.SD_CMD; no longer D1.SD_CMD
- net N$7: now also R10.1, U3.!RST; no longer R1.1, U5.!RST
- net N$8: now also D2.SD_DAT0; no longer D1.SD_DAT0
- net N$9: now also D2.SD_DAT1; no longer D1.SD_DAT1
- net NRF_CS: now also U2.P0.20, U5.IO5, U6.IO5; no longer U1.IO5, U2.IO5, U7.P0.20
- net NRF_LED0: now also R8.2, U2.P0.13; no longer R11.2, U7.P0.13
- net NRF_LED1: now also R9.2, U2.P0.14; no longer R12.2, U7.P0.14
- net NRF_LED2: now also R3.2, U2.P0.15; no longer R13.2, U7.P0.15
- net NRF_MISO: now also U2.P0.21, U5.IO19, U6.IO19; no longer U1.IO19, U2.IO19, U7.P0.21
- net NRF_MOSI: now also U2.P0.22, U5.IO23, U6.IO23; no longer U1.IO23, U2.IO23, U7.P0.22
- net NRF_SCLK: now also U2.P0.19, U5.IO18, U6.IO18; no longer U1.IO18, U2.IO18, U7.P0.19
- net RXD: now also U3.RXD; no longer U5.RXD
- net SD_HOST_CLK: now also D2.CLK, U5.IO14, U6.IO14; no longer D1.CLK, U1.IO14, U2.IO14
- net SD_HOST_CMD: now also D2.CMD, U5.IO15, U6.IO15; no longer D1.CMD, U1.IO15, U2.IO15
- net SD_HOST_D0: now also D2.DAT0, U5.IO2, U6.IO2; no longer D1.DAT0, U1.IO2, U2.IO2
- net SD_HOST_D1: now also D2.DAT1, U5.IO4, U6.IO4; no longer D1.DAT1, U1.IO4, U2.IO4
- net SD_HOST_D2: now also D2.DAT2, U5.IO12, U6.IO12; no longer D1.DAT2, U1.IO12, U2.IO12
- net SD_HOST_D3: now also D2.DAT3, U5.IO13, U6.IO13; no longer D1.DAT3, U1.IO13, U2.IO13
- net SWDCLK: now also J2.SWDCLK, U2.SWCLK; no longer J3.SWDCLK, U7.SWCLK
- net SWDIO: now also J2.SWDIO, U2.SWDIO; no longer J3.SWDIO, U7.SWDIO
- net TXD: now also U3.TXD; no longer U5.TXD
- net VBUS: now also C11.1, C3.1, C7.1, J3.+5V, U1.EN, U1.VIN, U3.VBUS, U3.VREGIN, U4.VUSB; no longer C1.1, C2.1, C5.1, J2.+5V, U3.EN, U3.VIN, U5.VBUS, U5.VREGIN, U6.VUSB
- net VCC: now also C12.1, C13.1, C5.1, D11.ANODE, D2.VCC, J2.VCC, R11.1, R13.2, U1.VOUT, U2.VDD, U2.VDDH, U3.VDD, U5.3V3, U5.EN, U6.3V3, U6.EN; no longer C11.1, C3.1, C7.1, D1.VCC, D2.ANODE, J3.VCC, R1.2, R9.1, U1.3V3, U1.EN, U2.3V3, U2.EN, U3.VOUT, U5.VDD, U7.VDD, U7.VDDH

Commit message: leave gpio12 floating, add diode
Parts:
- added D12: BLUE, leds:LED0603
- added Q1: DMN32D2LDF, fets:DMN32D2LDF
- added R15, R16: 10k, passives:RESISTOR0402_RES
- added R17, R18: 1k, passives:RESISTOR0402_RES
- added S1: B3U-1000P, switches:B3U-1000P
- added S3: JS202011CQN, switches:JS202011CQN
- D10, D4, D6: value YELLOW -> RED; DIGIKEY 160-1831-1-ND -> 160-1830-1-ND; MPN LTST-C193KSKT-5A -> LTST-C193KRKT-5A
- D11, D7: value BLUE -> YELLOW; DIGIKEY 160-1827-1-ND -> 160-1831-1-ND; MPN LTST-C193TBKT-5A -> LTST-C193KSKT-5A
- D2: value EMIF06-MSD01F2 -> (none); device passives:EMIF06-MSD01F2 -> passives:DIODE_ZENER0201; DIGIKEY (none) -> ESD7381MUT5GOSCT-ND; MPN (none) -> ESD7381MUT5G
- D3: value RED -> EMIF06-MSD01F2; device leds:LED0603 -> passives:EMIF06-MSD01F2; DIGIKEY 160-1830-1-ND -> (none); MPN LTST-C193KRKT-5A -> (none)
- D5: value RED -> YELLOW; DIGIKEY 160-1830-1-ND -> 160-1831-1-ND; MPN LTST-C193KRKT-5A -> LTST-C193KSKT-5A
- D9: value RED -> BLUE; DIGIKEY 160-1830-1-ND -> 160-1827-1-ND; MPN LTST-C193KRKT-5A -> LTST-C193TBKT-5A
- S2: value JS202011CQN -> B3U-1000P; device switches:JS202011CQN -> switches:B3U-1000P
Connections:
- removed net !RESET: J2.!RESET, U2.P0.18/RESET
- removed net N$10: D2.SD_DAT2, J1.DATA2/NC
- new net !NRF_RESET: J2.!RESET, U2.P0.18/RESET, U5.IO22, U6.IO22
- new net EN: R15.1, S1.P$2, U5.EN, U6.EN
- new net IO0: Q1.D1, U5.IO0, U6.IO0
- new net N$1: Q1.G1, R17.2
- new net N$4: Q1.G2, R18.2
- new net N$5: R16.2, R17.1, R18.1, S2.P$2
- net ESP32_0_RXD: now also S3.A2; no longer S2.A2
- net ESP32_0_TXD: now also S3.A1; no longer S2.A1
- net ESP32_1_RXD: now also S3.B2; no longer S2.B2
- net ESP32_1_TXD: now also S3.B1; no longer S2.B1
- net GND: now also D2.ANODE, D3.VSS, Q1.S, R16.1, S1.P$1; no longer D2.VSS
- net N$11: now also D3.SD_DAT3; no longer D2.SD_DAT3
- net N$12: now also D4.CATHODE; no longer D3.CATHODE
- net N$13: now also D3.SD_CLK; no longer D2.SD_CLK
- net N$14: now also D5.CATHODE; no longer D4.CATHODE
- net N$15: now also D8.CATHODE; no longer D7.CATHODE
- net N$19: now also D6.CATHODE; no longer D5.CATHODE
- net N$20: now also D7.CATHODE; no longer D6.CATHODE
- net N$21: now also D9.CATHODE; no longer D8.CATHODE
- net N$22: now also D10.CATHODE; no longer D9.CATHODE
- net N$23: now also D11.CATHODE; no longer D10.CATHODE
- net N$24: now also D12.CATHODE; no longer D11.CATHODE
- net N$6: now also D3.SD_CMD; no longer D2.SD_CMD
- net N$8: now also D3.SD_DAT0; no longer D2.SD_DAT0
- net N$9: now also D3.SD_DAT1; no longer D2.SD_DAT1
- net RXD: now also S3.I2; no longer S2.I2
- net SD_HOST_CLK: now also D3.CLK; no longer D2.CLK
- net SD_HOST_CMD: now also D3.CMD; no longer D2.CMD
- net SD_HOST_D0: now also D3.DAT0, Q1.D2; no longer D2.DAT0
- net SD_HOST_D1: now also D3.DAT1; no longer D2.DAT1
- net SD_HOST_D2: now also D2.CATHODE, J1.DATA2/NC; no longer D2.DAT2
- net SD_HOST_D3: now also D3.DAT3; no longer D2.DAT3
- net TXD: now also S3.I1; no longer S2.I1
- net VCC: now also D12.ANODE, D3.VCC, R15.2, S2.P$1; no longer D2.VCC, D3.ANODE, U5.EN, U6.EN
Other:
- moved on the sheet: C13, D1, D10, D11, D4, D5, D6, D7, D8, J1, R11
